Commit message: spawns thruster. Tinkered with bridges, not spinning

File: vrx_urdf/catamaran_description/custom_wamv/example_thruster_config.xacro (robot description, xacro)
@@ -5,10 +5,6 @@
       <xacro:engine prefix="left" position="-2.373776 1.027135 0.318237" orientation="0.0 0.0 0.0" />
       <xacro:engine prefix="right" position="-2.373776 -1.027135 0.318237" orientation="0.0 0.0 0.0" />
-      <xacro:engine prefix="forward_left" position="1 1.027135 0.318237" orientation="0.0 0.0 -1.07" />
-      <xacro:engine prefix="forward_right" position="1 -1.027135 0.318237" orientation="0.0 0.0 1.07" />
       <xacro:include filename="$(find wamv_gazebo)/urdf/thruster_layouts/wamv_gazebo_thruster_config.xacro" />
         <xacro:wamv_gazebo_thruster_config name="left" />
         <xacro:wamv_gazebo_thruster_config name="right" />
-        <xacro:wamv_gazebo_thruster_config name="forward_left" />
-        <xacro:wamv_gazebo_thruster_config name="forward_right" />
 </robot>

File: vrx_urdf/catamaran_description/custom_wamv/wamv_target.urdf (robot description, URDF)
Before this commit: robot WAM-V, 29 links, 28 joints
Links:
- removed link wamv/far_left_camera_link
- removed link wamv/far_left_camera_link_optical
- removed link wamv/far_left_camera_post_arm_link
- removed link wamv/far_left_camera_post_link
- removed link wamv/forward_left_engine_link
- removed link wamv/forward_left_propeller_link
- removed link wamv/forward_right_engine_link
- removed link wamv/forward_right_propeller_link
- removed link wamv/front_left_camera_link
- removed link wamv/front_left_camera_link_optical
- removed link wamv/front_left_camera_post_arm_link
- removed link wamv/front_left_camera_post_link
- removed link wamv/front_right_camera_link
- removed link wamv/front_right_camera_link_optical
- removed link wamv/front_right_camera_post_arm_link
- removed link wamv/front_right_camera_post_link
- removed link wamv/gps_wamv_link
- removed link wamv/imu_wamv_link
- removed link wamv/lidar_wamv_link
- removed link wamv/lidar_wamv_post_arm_link
- removed link wamv/lidar_wamv_post_link
Joints:
- removed joint wamv/base_to_far_left_camera_post_joint
- removed joint wamv/base_to_front_left_camera_post_joint
- removed joint wamv/base_to_front_right_camera_post_joint
- removed joint wamv/base_to_lidar_wamv_post_joint
- removed joint wamv/far_left_camera_post_arm_to_far_left_camera_joint
- removed joint wamv/far_left_camera_post_to_far_left_camera_post_arm_joint
- removed joint wamv/far_left_camera_to_far_left_camera_link_optical_joint
- removed joint wamv/forward_left_chassis_engine_joint
- removed joint wamv/forward_left_engine_propeller_joint
- removed joint wamv/forward_right_chassis_engine_joint
- removed joint wamv/forward_right_engine_propeller_joint
- removed joint wamv/front_left_camera_post_arm_to_front_left_camera_joint
- removed joint wamv/front_left_camera_post_to_front_left_camera_post_arm_joint
- removed joint wamv/front_left_camera_to_front_left_camera_link_optical_joint
- removed joint wamv/front_right_camera_post_arm_to_front_right_camera_joint
- removed joint wamv/front_right_camera_post_to_front_right_camera_post_arm_joint
- removed joint wamv/front_right_camera_to_front_right_camera_link_optical_joint
- removed joint wamv/gps_wamv_joint
- removed joint wamv/imu_wamv_joint
- removed joint wamv/lidar_wamv_post_arm_to_lidar_wamv_joint
- removed joint wamv/lidar_wamv_post_to_lidar_wamv_post_arm_joint
